File: _autosave-patch.kicad_sch (KiCad schematic)
At the start: 45 parts, among them J1 Conn_01x03, J2 Conn_01x16, J3 Conn_Coaxial_Small, J4 Conn_01x01, J5 Conn_01x01, J6 Conn_01x01, Q1 NMOS, SW1 SW_SPST, U1 74AHC1G08, U2 W25Q12NEZPIG

Commit message: Need to fix rst, ldo vbat and check parity
Parts:
- R10: value 10k -> 100k
Changed lines of the file:
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@@
 			)
 		)
-		(property "Value" "10k"
+		(property "Value" "100k"
 			(at 170.18 43.1801 0)
 			(show_name no)
