File: patch.kicad_sch (KiCad schematic)
At the start: 45 parts, among them J1 Conn_01x03, J2 Conn_01x16, J3 Conn_Coaxial_Small, J4 Conn_01x01, J5 Conn_01x01, J6 Conn_01x01, Q1 NMOS, SW1 SW_SPST, U1 74AHC1G08, U2 W25Q12NEZPIG

Commit message: Corrected connection
Parts:
- R10: value 10k -> 100k
Connections:
- net GND: no longer J2.5 (Pin_5)
- net LDO_VBAT: now also J2.5 (Pin_5); no longer J2.4 (Pin_4)
- net UART.RX: now also J2.3 (Pin_3); no longer J2.2 (Pin_2)
- net UART.TX: now also J2.4 (Pin_4); no longer J2.3 (Pin_3)
- net nRST: now also J2.2 (Pin_2)
Changed lines of the file:
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@@
 	(wire
 		(pts
+			(xy 124.46 52.07) (xy 121.92 52.07)
+		)
+		(stroke
+			(width 0)
+			(type default)
+		)
+	)
+	(wire
+		(pts
 			(xy 173.99 92.71) (xy 171.45 92.71)
 		)
@@
 	(wire
 		(pts
-			(xy 124.46 34.29) (xy 124.46 58.42)
-		)
-		(stroke
-			(width 0)
-			(type default)
-		)
-	)
-	(wire
-		(pts
 			(xy 97.79 186.69) (xy 100.33 182.88)
 		)
@@
 	(wire
 		(pts
-			(xy 121.92 34.29) (xy 121.92 58.42)
-		)
-		(stroke
-			(width 0)
-			(type default)
-		)
-	)
-	(wire
-		(pts
 			(xy 50.8 166.37) (xy 66.04 166.37)
 		)
@@
 	(wire
 		(pts
+			(xy 121.92 34.29) (xy 121.92 50.8)
+		)
+		(stroke
+			(width 0)
+			(type default)
+		)
+	)
+	(wire
+		(pts
 			(xy 247.65 147.32) (xy 271.78 147.32)
 		)
@@
 	(wire
 		(pts
+			(xy 124.46 58.42) (xy 124.46 53.34)
+		)
+		(stroke
+			(width 0)
+			(type default)
+		)
+	)
+	(wire
+		(pts
 			(xy 33.02 99.06) (xy 33.02 96.52)
 		)
@@
 	(wire
 		(pts
+			(xy 127 58.42) (xy 127 54.61)
+		)
+		(stroke
+			(width 0)
+			(type default)
+		)
+	)
+	(wire
+		(pts
 			(xy 184.15 128.27) (xy 184.15 127)
 		)
@@
 	(wire
 		(pts
-			(xy 165.1 40.64) (xy 172.72 40.64)
+			(xy 121.92 52.07) (xy 121.92 58.42)
 		)
 		(stroke
@@
 	(wire
 		(pts
-			(xy 127 34.29) (xy 127 58.42)
+			(xy 165.1 40.64) (xy 172.72 40.64)
 		)
 		(stroke
@@
 	(wire
 		(pts
+			(xy 127 54.61) (xy 129.54 54.61)
+		)
+		(stroke
+			(width 0)
+			(type default)
+		)
+	)
+	(wire
+		(pts
 			(xy 40.64 184.15) (xy 40.64 185.42)
 		)
@@
 	(wire
 		(pts
+			(xy 124.46 53.34) (xy 127 53.34)
+		)
+		(stroke
+			(width 0)
+			(type default)
+		)
+	)
+	(wire
+		(pts
 			(xy 137.16 34.29) (xy 137.16 58.42)
 		)
@@
 	(wire
 		(pts
+			(xy 127 34.29) (xy 127 53.34)
+		)
+		(stroke
+			(width 0)
+			(type default)
+		)
+	)
+	(wire
+		(pts
 			(xy 58.42 176.53) (xy 67.31 176.53)
 		)
@@
 	(wire
 		(pts
+			(xy 129.54 34.29) (xy 129.54 54.61)
+		)
+		(stroke
+			(width 0)
+			(type default)
+		)
+	)
+	(wire
+		(pts
 			(xy 121.92 124.46) (xy 121.92 119.38)
 		)
@@
 	(wire
 		(pts
+			(xy 124.46 34.29) (xy 124.46 52.07)
+		)
+		(stroke
+			(width 0)
+			(type default)
+		)
+	)
+	(wire
+		(pts
 			(xy 25.4 83.82) (xy 25.4 86.36)
 		)
@@
 	)
 	(label "LDO_VBAT"
-		(at 127 52.07 90)
+		(at 129.54 52.07 90)
 		(effects
 			(font
@@
 		)
 	)
+	(label "nRST"
+		(at 121.92 50.8 90)
+		(effects
+			(font
+				(size 1.27 1.27)
+			)
+			(justify left bottom)
+		)
+	)
 	(label "GND"
 		(at 176.53 134.62 0)
@@
 	)
 	(label "UART.TX"
-		(at 124.46 52.07 90)
+		(at 127 52.07 90)
 		(effects
 			(font
@@
 	)
 	(label "UART.RX"
-		(at 121.92 52.07 90)
+		(at 124.46 52.07 90)
 		(effects
 			(font
@@
 	)
 	(symbol
-		(lib_id "power:GND")
-		(at 129.54 34.29 0)
-		(unit 1)
-		(body_style 1)
-		(exclude_from_sim no)
-		(in_bom yes)
-		(on_board yes)
-		(in_pos_files yes)
-		(dnp no)
-		(fields_autoplaced yes)
-		(property "Reference" "#PWR09"
-			(at 129.54 40.64 0)
-			(hide yes)
-			(show_name no)
-			(do_not_autoplace no)
-			(effects
-				(font
-					(size 1.27 1.27)
-				)
-			)
-		)
-		(property "Value" "GND"
-			(at 129.5401 38.1 90)
-			(hide yes)
-			(show_name no)
-			(do_not_autoplace no)
-			(effects
-				(font
-					(size 1.27 1.27)
-				)
-				(justify right)
-			)
-		)
-		(property "Footprint" ""
-			(at 129.54 34.29 0)
-			(hide yes)
-			(show_name no)
-			(do_not_autoplace no)
-			(effects
-				(font
-					(size 1.27 1.27)
-				)
-			)
-		)
-		(property "Datasheet" ""
-			(at 129.54 34.29 0)
-			(hide yes)
-			(show_name no)
-			(do_not_autoplace no)
-			(effects
-				(font
-					(size 1.27 1.27)
-				)
-			)
-		)
-		(property "Description" "Power symbol creates a global label with name \"GND\" , ground"
-			(at 129.54 34.29 0)
-			(hide yes)
-			(show_name no)
-			(do_not_autoplace no)
-			(effects
-				(font
-					(size 1.27 1.27)
-				)
-			)
-		)
-		(pin "1"
-		)
-		(instances
-			(project "patch"
-				(path "/3aa5b069-cd8a-454c-b0f9-98fe40d88006"
-					(reference "#PWR09")
-					(unit 1)
-				)
-			)
-		)
-	)
-	(symbol
 		(lib_id "QFN64-scoket:264-5205-01")
 		(at 115.57 63.5 0)
@@
 			)
 		)
-		(property "Value" "10k"
+		(property "Value" "100k"
 			(at 170.18 43.1801 0)
 			(show_name no)
