File: patch-backups/patch-2026-07-28_184002/patch.kicad_sch (KiCad schematic)
At the start: 45 parts, among them J1 Conn_01x03, J2 Conn_01x16, J3 Conn_Coaxial_Small, J4 Conn_01x01, J5 Conn_01x01, J6 Conn_01x01, Q1 NMOS, SW1 SW_SPST, U1 74AHC1G08, U2 W25Q12NEZPIG

Commit message: Need to fix rst, ldo vbat and check parity
Parts:
- removed C14: 100n, Capacitor_SMD:C_0603_1608Metric, symbol Device:C_Small
- removed Crect1: 1u, Capacitor_SMD:C_0603_1608Metric, symbol Device:C_Small
- removed Ctune1: 10u, Capacitor_SMD:C_0603_1608Metric, symbol Device:C_Small
- removed D4: D_Schottky, Diode_SMD:D_0603_1608Metric, symbol Device:D_Schottky
- removed NT1: NetTie_2, libs:1MHz_coil_29x14, symbol Device:NetTie_2
- removed R10, R11, R12, R13, R14, R15, R16: 10k, Resistor_SMD:R_0603_1608Metric, symbol Device:R_US
- removed Rchg1: 1k, Resistor_SMD:R_0603_1608Metric, symbol Device:R_US
- removed SW1: SW_SPST, libs:SPST_1.6x3mm, symbol Switch:SW_SPST
- removed U2: W25Q12NEZPIG, Package_SO:SOIC-8_5.23x5.23mm_P1.27mm, symbol Memory_Flash:W25Q16JVSS
- R5, R6, R7: value 330 -> 10k
Connections:
- net LDO_VBAT: no longer HEEPidermis1.13, HEEPidermis1.62, J2.4 (Pin_4)
- new net SUPPLY_IO_VDD: HEEPidermis1.13, HEEPidermis1.62, J2.4 (Pin_4)
Other:
- note removed: "Connector for programming"
- note removed: "Flash for storage"
- note removed: "LED for debug"
- note removed: "LEDs from dLC"
- note removed: "Pushbutton to sleep/wake-up"
- note removed: "Radio modulation"
- note removed: "WPT for battery charging"
- moved on the sheet: D2, D3, R6, R7
