File: patch-backups/patch-2026-08-07_195143/patch.kicad_sch (KiCad schematic)
At the start: 45 parts, among them J1 Conn_01x03, J2 Conn_01x16, J3 Conn_Coaxial_Small, J4 Conn_01x01, J5 Conn_01x01, J6 Conn_01x01, Q1 NMOS, SW1 SW_SPST, U1 74AHC1G08, U2 W25Q12NEZPIG

Commit message: Need to fix rst, ldo vbat and check parity
Parts:
- removed C14: 100n, Capacitor_SMD:C_0603_1608Metric, symbol Device:C_Small
- removed NT1: NetTie_2, libs:1MHz_coil_29x14, symbol Device:NetTie_2
- removed R11, R12, R13, R14, R15, R16: 10k, Resistor_SMD:R_0603_1608Metric, symbol Device:R_US
- removed U2: W25Q12NEZPIG, Package_SO:SOIC-8_5.23x5.23mm_P1.27mm, symbol Memory_Flash:W25Q16JVSS
- R5, R6, R7: value 330 -> 10k
- SW1: footprint libs:SPST_1.6x3mm -> Button_Switch_SMD:SW_SPST_FSMSM
Connections:
- net LDO_VBAT: no longer HEEPidermis1.13, HEEPidermis1.62, J2.4 (Pin_4)
- net at R10.1, SW1.1 (A): no longer HEEPidermis1.49, R5.2
- net ANT renamed ant_p
- new net: HEEPidermis1.49, R5.2
- new net SUPPLY_IO_VDD: HEEPidermis1.13, HEEPidermis1.62, J2.4 (Pin_4)
Other:
- note added: "(!) Add a pushbuttom to send the system to sleep"
- note added: "(!) Add an external flash just in case"
- note added: "(!) Choose these values correctly"
- note added: "(!) Footprint for 1MHz clock"
- note added: "(!) WPT for battery charging"
- note removed: "Connector for programming"
- note removed: "Flash for storage"
- note removed: "LED for debug"
- note removed: "LEDs from dLC"
- note removed: "Pushbutton to sleep/wake-up"
- note removed: "Radio modulation"
- note removed: "WPT for battery charging"
